Commit message: 変更

File: models/robot.urdf (robot description, URDF)
Before this commit: robot so101_new_calib, 8 links, 7 joints
Joints:
- joint elbow_flex: limit lower=-1.69 upper=1.69 effort=10 velocity=10 -> lower=-3.14 upper=3.14 effort=10 velocity=10
- joint shoulder_lift: limit lower=-1.74533 upper=1.74533 effort=10 velocity=10 -> lower=-3.14159 upper=3.14159 effort=10 velocity=10
- joint shoulder_pan: limit lower=-1.91986 upper=1.91986 effort=10 velocity=10 -> lower=-3.14159 upper=3.14159 effort=10 velocity=10
- joint wrist_flex: limit lower=-1.65806 upper=1.65806 effort=10 velocity=10 -> lower=-3.14 upper=3.14 effort=10 velocity=10
- joint wrist_roll: limit lower=-2.74385 upper=2.84121 effort=10 velocity=10 -> lower=-3.14 upper=3.14 effort=10 velocity=10

Commit message: 実機とシミュレーション使い分けれるように変更

File: models/robot.urdf (robot description, URDF)
Before this commit: robot so101_new_calib, 8 links, 7 joints
Links:
- added link world
Joints:
- added joint world_to_base: type fixed, parent world, child base_link, origin xyz=0 0 0.5 rpy=0 0 0
